File: proteus-mitsubishi76-adapter.kicad_pcb (KiCad board)
At the start: 2 copper layers, 149 x 157.5 mm, 5 parts, among them J1 TE-3-178780-6

Commit message: Upd sch
Parts:
- added BRD1: proteus, kicad6-libraries:proteus, F.Cu at (286.6, 94.7)
- added D1: D_Schottky, Diode_SMD:D_SMA, F.Cu at (515.9, 89.5)
- added D2: DNP, Diode_SMD:D_SMA, F.Cu at (511.3, 97.8)
- added D3: D_Schottky, Diode_SMD:D_SMA, F.Cu at (503.3, 102.3)
- added D4: D_Schottky, Diode_SMD:D_SMA, F.Cu at (427.6, 179.0)
- added D5: D_Schottky, Diode_SMD:D_SMA, F.Cu at (419.6, 179.0)
- added D6: D_Schottky, Diode_SMD:D_SMA, F.Cu at (503.3, 97.8)
- added D7: D_Schottky, Diode_SMD:D_SMA, F.Cu at (529.9, 81.2)
- added F1: Fuse-Pad-Pad, hellen-one-common:PAD-1206-PAD, F.Cu at (367.0, 183.6)
- added F2: Fuse-Pad-Pad, hellen-one-common:PAD-1206-PAD, F.Cu at (375.0, 183.6)
- added F3: Fuse-Pad-Pad, hellen-one-common:PAD-1206-PAD, F.Cu at (383.0, 183.6)
- added G1: RUSEFI_LOGO, kicad6-libraries:rusefi_logo, F.Cu at (543.7, 74.7)
- added G2: PROTO_AREA, hellen-one-common:PROTO_AREA, F.Cu at (394.0, 170.1)
- added G3: PROTO_AREA, hellen-one-common:PROTO_AREA, F.Cu at (394.0, 178.3)
- added G4: PROTO_AREA, hellen-one-common:PROTO_AREA, F.Cu at (500.8, 80.5)
- added G5: PROTO_AREA, hellen-one-common:PROTO_AREA, F.Cu at (495.7, 165.3)
- added G6: PROTO_AREA, hellen-one-common:PROTO_AREA, F.Cu at (541.4, 64.2)
- added G7: PROTO_AREA, hellen-one-common:PROTO_AREA, F.Cu at (407.3, 170.1)
- added G8: PROTO_AREA, hellen-one-common:PROTO_AREA, F.Cu at (514.1, 80.5)
- added J2: TE-3-178780-6, kicad6-libraries:TE-3-178780-6, F.Cu at (157.0, 71.6)
- added J4: Conn_01x06, Connector_PinHeader_2.54mm:PinHeader_1x06_P2.54mm_Vertical, F.Cu at (496.4, 148.7)
- added J5: Conn_01x01, TestPoint:TestPoint_Pad_D4.0mm, F.Cu at (448.4, 174.4)
- added M1: Module-wbo-0.3, hellen-one-wbo-0.3:wbo, F.Cu at (200.3, 196.4)
- added M2: Module-can-0.1, hellen-one-can-0.1:can, F.Cu at (500.0, 94.8)
- added P1: Pad, hellen-one-common:PAD-TH, F.Cu at (535.8, 80.8)
- added P10: Pad, hellen-one-common:PAD-TH, F.Cu at (522.0, 108.0)
- added P11: Pad, hellen-one-common:PAD-TH, F.Cu at (518.2, 114.3)
- added P12: Pad, hellen-one-common:PAD-TH, F.Cu at (501.1, 131.2)
- added P13: Pad, hellen-one-common:PAD-TH, F.Cu at (507.3, 131.2)
- added P14: Pad, hellen-one-common:PAD-TH, F.Cu at (553.2, 76.5)
- added P15: Pad, hellen-one-common:PAD-TH, F.Cu at (454.4, 177.6)
- added P16: Pad, hellen-one-common:PAD-TH, F.Cu at (514.5, 110.5)
- added P17: Pad, hellen-one-common:PAD-TH, F.Cu at (548.6, 84.1)
- added P18: Pad, hellen-one-common:PAD-TH, F.Cu at (564.9, 68.3)
- added P19: Pad, hellen-one-common:PAD-TH, F.Cu at (557.0, 72.7)
- added P2: Pad, hellen-one-common:PAD-TH, F.Cu at (541.7, 80.3)
- added P20: Pad, hellen-one-common:PAD-TH, F.Cu at (446.9, 179.3)
- added P21: Pad, hellen-one-common:PAD-TH, F.Cu at (553.2, 72.7)
- added P22: Pad, hellen-one-common:PAD-TH, F.Cu at (537.5, 92.0)
- added P23: Pad, hellen-one-common:PAD-TH, F.Cu at (512.5, 121.8)
- added P24: Pad, hellen-one-common:PAD-TH, F.Cu at (535.2, 101.5)
- added P25: Pad, hellen-one-common:PAD-TH, F.Cu at (549.4, 76.5)
- added P26: Pad, hellen-one-common:PAD-TH, F.Cu at (508.7, 126.4)
- added P27: Pad, hellen-one-common:PAD-TH, F.Cu at (552.4, 84.1)
- added P28: Pad, hellen-one-common:PAD-TH, F.Cu at (507.8, 115.0)
- added P29: Pad, hellen-one-common:PAD-TH, F.Cu at (568.7, 64.5)
- added P3: Pad, hellen-one-common:PAD-TH, F.Cu at (531.5, 97.7)
- added P30: Pad, hellen-one-common:PAD-TH, F.Cu at (572.5, 64.5)
- added P31: Pad, hellen-one-common:PAD-TH, F.Cu at (447.9, 183.1)
- added P32: Pad, hellen-one-common:PAD-TH, F.Cu at (539.0, 95.8)
- added P33: Pad, hellen-one-common:PAD-TH, F.Cu at (504.9, 123.6)
- added P34: Pad, hellen-one-common:PAD-TH, F.Cu at (533.7, 93.9)
- added P35: Pad, hellen-one-common:PAD-TH, F.Cu at (549.4, 72.7)
- added P36: Pad, hellen-one-common:PAD-TH, F.Cu at (549.4, 80.3)
- added P37: Pad, hellen-one-common:PAD-TH, F.Cu at (522.0, 111.8)
- added P38: Pad, hellen-one-common:PAD-TH, F.Cu at (514.5, 114.3)
- added P39: Pad, hellen-one-common:PAD-TH, F.Cu at (508.7, 122.6)
- added P4: Pad, hellen-one-common:PAD-TH, F.Cu at (450.6, 179.3)
- added P40: Pad, hellen-one-common:PAD-TH, F.Cu at (535.1, 88.2)
- added P41: Pad, hellen-one-common:PAD-TH, F.Cu at (531.5, 101.5)
- added P42: Pad, hellen-one-common:PAD-TH, F.Cu at (518.2, 110.5)
- added P43: Pad, hellen-one-common:PAD-TH, F.Cu at (444.1, 183.1)
- added P44: Pad, hellen-one-common:PAD-TH, F.Cu at (538.9, 88.2)
- added P45: Pad, hellen-one-common:PAD-TH, F.Cu at (453.3, 173.2)
- added P46: Pad, hellen-one-common:PAD-TH, F.Cu at (541.3, 92.0)
- added P47: Pad, hellen-one-common:PAD-TH, F.Cu at (542.7, 87.9)
- added P48: Pad, hellen-one-common:PAD-TH, F.Cu at (541.1, 84.1)
- added P49: Pad, hellen-one-common:PAD-TH, F.Cu at (457.1, 173.8)
- added P5: Pad, hellen-one-common:PAD-TH, F.Cu at (521.1, 104.2)
- added P50: Pad, hellen-one-common:PAD-TH, F.Cu at (501.1, 127.4)
- added P51: Pad, hellen-one-common:PAD-TH, F.Cu at (515.4, 118.1)
- added P52: Pad, hellen-one-common:PAD-TH, F.Cu at (527.7, 100.5)
- added P53: Pad, hellen-one-common:PAD-TH, F.Cu at (528.7, 105.3)
- added P54: Pad, hellen-one-common:PAD-TH, F.Cu at (458.2, 177.6)
- added P55: Pad, hellen-one-common:PAD-TH, F.Cu at (568.7, 68.3)
- added P56: Pad, hellen-one-common:PAD-TH, F.Cu at (557.0, 76.5)
- added P57: Pad, hellen-one-common:PAD-TH, F.Cu at (523.9, 100.5)
- added P58: Pad, hellen-one-common:PAD-TH, F.Cu at (544.9, 84.1)
- added P59: Pad, hellen-one-common:PAD-TH, F.Cu at (388.9, 183.9)
- added P6: Pad, hellen-one-common:PAD-TH, F.Cu at (524.9, 104.2)
- added P60: Pad, hellen-one-common:PAD-TH, F.Cu at (507.8, 118.8)
- added P61: Pad, hellen-one-common:PAD-TH, F.Cu at (546.5, 87.9)
- added P62: Pad, hellen-one-common:PAD-TH, F.Cu at (501.1, 123.6)
- added P63: Pad, hellen-one-common:PAD-TH, F.Cu at (511.6, 118.1)
- added P64: Pad, hellen-one-common:PAD-TH, F.Cu at (501.1, 134.9)
- added P65: Pad, hellen-one-common:PAD-TH, F.Cu at (451.6, 183.1)
- added P66: Pad, hellen-one-common:PAD-TH, F.Cu at (564.9, 64.5)
- added P67: Pad, hellen-one-common:PAD-TH, F.Cu at (535.2, 97.7)
- added P7: Pad, hellen-one-common:PAD-TH, F.Cu at (564.9, 72.0)
- added P8: Pad, hellen-one-common:PAD-TH, F.Cu at (545.5, 80.3)
- added P9: Pad, hellen-one-common:PAD-TH, F.Cu at (504.9, 127.4)
- added Q1: AUIPS2041LTR, Package_TO_SOT_SMD:SOT-223, F.Cu at (433.8, 172.6)
- added Q2: AUIPS2041LTR, Package_TO_SOT_SMD:SOT-223, F.Cu at (558.1, 66.7)
- added Q3: AUIPS2041LTR, Package_TO_SOT_SMD:SOT-223, F.Cu at (410.6, 180.9)
- added Q4: AUIPS2041LTR, Package_TO_SOT_SMD:SOT-223, F.Cu at (423.9, 172.6)
- added R1: Jumper-Pad-Pad, hellen-one-common:PAD-0805-PAD, F.Cu at (535.9, 84.9)
- added R10: Jumper-Pad-Pad, hellen-one-common:PAD-0805-PAD, F.Cu at (502.6, 120.3)
- added R11: Jumper-Pad-Pad, hellen-one-common:PAD-0805-PAD, F.Cu at (515.2, 93.2)
- added R12: Jumper-Pad-Pad, hellen-one-common:PAD-0805-PAD, F.Cu at (438.9, 183.9)
- added R13: Jumper-Pad-Pad, hellen-one-common:PAD-0805-PAD, F.Cu at (529.9, 87.8)
- added R14: Jumper-Pad-Pad, hellen-one-common:PAD-0805-PAD, F.Cu at (502.6, 117.4)
- added R15: Jumper-Pad-Pad, hellen-one-common:PAD-0805-PAD, F.Cu at (502.6, 106.0)
- added R16: Jumper-Pad-Pad, hellen-one-common:PAD-0805-PAD, F.Cu at (529.9, 90.6)
- added R17: Jumper-Pad-Pad, hellen-one-common:PAD-0805-PAD, F.Cu at (502.6, 108.9)
- added R18: Jumper-Pad-Pad, hellen-one-common:PAD-0805-PAD, F.Cu at (525.3, 97.2)
- added R19: Jumper-Pad-Pad, hellen-one-common:PAD-0805-PAD, F.Cu at (515.9, 107.2)
- added R2: Jumper-Pad-Pad, hellen-one-common:PAD-0805-PAD, F.Cu at (529.2, 84.9)
- added R20: Jumper-Pad-Pad, hellen-one-common:PAD-0805-PAD, F.Cu at (435.0, 178.2)
- added R21: Jumper-Pad-Pad, hellen-one-common:PAD-0805-PAD, F.Cu at (502.6, 111.7)
- added R22: Jumper-Pad-Pad, hellen-one-common:PAD-0805-PAD, F.Cu at (515.9, 104.3)
- added R23: Jumper-Pad-Pad, hellen-one-common:PAD-0805-PAD, F.Cu at (510.6, 101.5)
- added R24: Jumper-Pad-Pad, hellen-one-common:PAD-0805-PAD, F.Cu at (528.5, 94.3)
- added R25: Jumper-Pad-Pad, hellen-one-common:PAD-0805-PAD, F.Cu at (435.0, 181.0)
- added R26: Jumper-Pad-Pad, hellen-one-common:PAD-0805-PAD, F.Cu at (442.1, 169.9)
- added R27: Jumper-Pad-Pad, hellen-one-common:PAD-0805-PAD, F.Cu at (502.6, 114.6)
- added R28: Jumper-Pad-Pad, hellen-one-common:PAD-0805-PAD, F.Cu at (448.7, 169.9)
- added R29: Jumper-Pad-Pad, hellen-one-common:PAD-0805-PAD, F.Cu at (509.2, 108.9)
- added R3: Jumper-Pad-Pad, hellen-one-common:PAD-0805-PAD, F.Cu at (441.7, 178.5)
- added R30: Jumper-Pad-Pad, hellen-one-common:PAD-0805-PAD, F.Cu at (418.9, 182.7)
- added R31: Jumper-Pad-Pad, hellen-one-common:PAD-0805-PAD, F.Cu at (521.9, 94.3)
- added R32: Jumper-Pad-Pad, hellen-one-common:PAD-0805-PAD, F.Cu at (442.1, 175.6)
- added R33: Jumper-Pad-Pad, hellen-one-common:PAD-0805-PAD, F.Cu at (518.7, 100.0)
- added R34: Jumper-Pad-Pad, hellen-one-common:PAD-0805-PAD, F.Cu at (425.6, 182.7)
- added R35: Jumper-Pad-Pad, hellen-one-common:PAD-0805-PAD, F.Cu at (432.2, 183.9)
- added R36: Jumper-Pad-Pad, hellen-one-common:PAD-0805-PAD, F.Cu at (502.1, 147.8)
- added R37: 10k, Resistor_SMD:R_0402_1005Metric, F.Cu at (439.8, 180.9)
- added R38: 10k, Resistor_SMD:R_0402_1005Metric, F.Cu at (456.4, 169.5)
- added R39: 10k, Resistor_SMD:R_0402_1005Metric, F.Cu at (453.5, 169.5)
- added R4: Jumper-Pad-Pad, hellen-one-common:PAD-0805-PAD, F.Cu at (442.1, 172.8)
- added R40: 10k, Resistor_SMD:R_0402_1005Metric, F.Cu at (459.3, 169.5)
- added R5: Jumper-Pad-Pad, hellen-one-common:PAD-0805-PAD, F.Cu at (509.2, 111.7)
- added R6: Jumper-Pad-Pad, hellen-one-common:PAD-0805-PAD, F.Cu at (523.3, 88.6)
- added R7: Jumper-Pad-Pad, hellen-one-common:PAD-0805-PAD, F.Cu at (509.2, 106.0)
- added R8: Jumper-Pad-Pad, hellen-one-common:PAD-0805-PAD, F.Cu at (518.7, 97.2)
- added R9: Jumper-Pad-Pad, hellen-one-common:PAD-0805-PAD, F.Cu at (523.3, 91.5)
- J1: value TE-3-178780-6 -> XH-10AW; footprint libs:TE-3-178780-6 -> Connector_JST:JST_XH_S10B-XH-A_1x10_P2.50mm_Horizontal
- moved J1 156.9 mm to (245.2, 201.8)
- moved H2 1.00 mm to (148.4, 210.1)
- moved H4 1.00 mm to (287.4, 210.1)
- moved H1 0.70 mm to (287.4, 78.9)
- moved H3 0.70 mm to (148.4, 78.9)
Connections:
- J1 pad 1: unconnected-(J1-Pad1) -> /12V_MR
- J1 pad 10: unconnected-(J1-Pad10) -> GND
- J1 pad 2: unconnected-(J1-Pad2) -> /12V_MR
- J1 pad 3: unconnected-(J1-Pad3) -> /WBO_Vs
- J1 pad 4: unconnected-(J1-Pad4) -> /WBO_Vs/Ip
- J1 pad 5: unconnected-(J1-Pad5) -> /WBO_Ip
- J1 pad 6: unconnected-(J1-Pad6) -> /WBO_R_Trim
- J1 pad 7: unconnected-(J1-Pad7) -> /WBO_H-
- J1 pad 8: unconnected-(J1-Pad8) -> /WBO_H-
- J1 pad 9: unconnected-(J1-Pad9) -> GND
Other:
- board size 149 x 157.5 mm -> 149 x 158 mm

Commit message: Board routing
Parts:
- added G***: LOGO, LOGO, B.Cu at (207.6, 130.3)
- moved G1 403.2 mm to (164.1, 210.7)
- moved P30 400.0 mm to (172.9, 83.1)
- moved P29 393.2 mm to (175.9, 83.1)
- moved P66 385.6 mm to (187.0, 141.3)
- moved G6 378.2 mm to (183.4, 186.1), turned to 180 degrees
- moved P32 375.8 mm to (163.4, 83.1)
- moved G8 371.9 mm to (163.4, 204.1), turned to 90 degrees
- moved P18 365.3 mm to (199.9, 83.1)
- moved P27 365.0 mm to (187.4, 83.1)
- moved R24 364.3 mm to (164.2, 91.1), turned to -90 degrees
- moved R31 362.9 mm to (159.0, 91.1), turned to -90 degrees
- moved P61 361.6 mm to (186.9, 126.1), turned to -90 degrees
- moved P34 360.9 mm to (172.9, 88.1)
- moved P19 360.2 mm to (196.9, 83.1)
- moved P36 357.4 mm to (206.4, 180.5)
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Routing:
- net /12V_MR: track 0.00 -> 179.1 mm, vias 0 -> 6
- net +5VA: track 0.00 -> 158.5 mm
- net /IN_CRANK: track 0.00 -> 104.2 mm
- net /IN_VAF: track 0.00 -> 102.6 mm, vias 0 -> 1
- net /OUT_MAIN_RELAY: track 0.00 -> 98.2 mm, vias 0 -> 2
- net /IN_CAM: track 0.00 -> 97.2 mm
- net /OUT_CHECK_ENGINE: track 0.00 -> 91.7 mm, vias 0 -> 2
- net /IN_VSS: track 0.00 -> 88.4 mm
- net /OUT_FUEL_PUMP_HI/LO_RELAY: track 0.00 -> 81.6 mm, vias 0 -> 1
- net /OUT_IDLE3: track 0.00 -> 79.3 mm
- net /IDLE4: track 0.00 -> 75.9 mm, vias 0 -> 1
- net /OUT_INJ6/TURBOCHRG_WG_SOLEOID: track 0.00 -> 73.1 mm, vias 0 -> 1
- net /12V_IGN: track 0.00 -> 71.8 mm
- net /OUT_INJ2: track 0.00 -> 71.1 mm
- net /IN_KNOCK: track 0.00 -> 67.2 mm
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- added copper zone on B.Cu, net GND
- added copper zone on F.Cu, net GND
Other:
- board text added: "Always looking for C/C++/PHP/Java developers https://rusefi.com/s/mission"
- board text added: "https://rusefi.com"
- board text added: "proteus-mitsubishi76-adapter"
- board text added: "rev 0.1"
